File: hardware/c3dpb.kicad_pcb (KiCad board)
At the start: 4 copper layers, 80 x 58.8 mm, 317 parts, among them IC1 TMC2209, IC2 TMC2209, IC3 TMC2209, IC4 TMC2209, J1 Conn_01x01, J10 Conn_01x04, J100 Conn_01x01, J101 Conn_01x01, J102 Conn_01x01, J11 Screw_Terminal_01x04, J12 Conn_01x03, J13 Conn_01x03, J14 Conn_01x03, J15 Conn_01x03, J16 Conn_01x03, J17 Conn_01x03, J18 Conn_01x03, J19 Conn_01x03, J2 Conn_01x01, J20 Conn_01x03, J21 Conn_01x03, J24 Conn_01x01, J3 Conn_01x01, J39 Screw_Terminal_01x02, J4 Conn_01x01, J44 Conn_01x01, J45 Conn_01x01, J48 Conn_01x01, J49 Conn_01x01, J5 Conn_01x01, J50 Conn_01x01, J51 Conn_01x01, J53 Conn_01x01, J54 Conn_01x01, J55 Conn_01x01, J56 Conn_01x01, J57 Conn_01x01, J58 Conn_01x01, J59 Conn_01x01, J6 Conn_01x01, J60 USB_C_Receptacle, J62 Conn_01x02, J68 Conn_01x01, J69 Conn_01x01, J7 Conn_01x04, J70 Conn_01x01, J71 Conn_01x02, J72 Conn_01x02, J73 Conn_01x02, J8 Conn_01x04, J9 Conn_01x04, J94 Conn_01x01, J95 Conn_01x01, J96 Conn_01x01, J98 Conn_01x01, J99 Conn_01x01, Q1 AON7418, Q10 AO3402, Q11 AO3402, Q12 AO3402, Q13 AO3402, Q14 AO3402, Q2 AO3400, Q3 AO3402, Q4 AON7418, Q5 AON7418, Q6 AO3402, Q7 AO3402, Q8 AO3402, Q9 AO3402, SW1 3x6mm, U1 ATSAMD51J19A-M, U2 LM1117-3.3, U3 SY8303, U4 SY8303, U5 MAX6675, U6 IR4427S

Commit message: new con
Parts:
- added C76: 4.7u, _Generic:0805_CAP, F.Cu at (129.4, 45.1)
- added C77: 4.7u, _Generic:0805_CAP, F.Cu at (150.7, 45.1)
- added D16: 3.6v, _Generic:SOD-523_DIODE, F.Cu at (144.3, 37.1)
- added D17: 3.6v, _Generic:SOD-523_DIODE, F.Cu at (157.0, 44.9)
- added J22: Conn_01x03, _Generic:JST_XH_3P, F.Cu at (164.9, 55.0)
- added J23: Conn_01x03, _Generic:JST_XH_3P, F.Cu at (134.3, 65.7)
- added JP34: SolderJumper_2_Open, _Generic:Solder Jumper 2P, F.Cu at (138.2, 44.8)
- added JP35: SolderJumper_2_Open, _Generic:Solder Jumper 2P, F.Cu at (143.8, 38.9)
- added JP36: SolderJumper_4_Open, _Generic:SolderJumper_JST, F.Cu at (141.2, 38.4)
- added JP37: SolderJumper_2_Open, _Generic:Solder Jumper 2P, F.Cu at (159.5, 44.8)
- added JP38: SolderJumper_2_Open, _Generic:Solder Jumper 2P, F.Cu at (165.1, 38.9)
- added JP39: SolderJumper_4_Open, _Generic:SolderJumper_JST, F.Cu at (162.5, 38.4)
- added Q15: AO3402, _Generic:SOT-23, F.Cu at (141.5, 42.7)
- added Q16: AO3402, _Generic:SOT-23, F.Cu at (162.8, 42.7)
- added R53: 4.7k, _Generic:0603_RES, F.Cu at (135.7, 44.9)
- added R54: 1meg, _Generic:0603_RES, F.Cu at (132.7, 44.9)
- added R55: 4.7k, _Generic:0603_RES, F.Cu at (154.0, 44.9)
- added R56: 1meg, _Generic:0603_RES, F.Cu at (165.6, 37.1)
- moved J17 161.2 mm to (140.7, 65.7), turned to 270 degrees
- moved J13 139.8 mm to (139.6, 55.0), turned to 90 degrees
- moved J20 134.5 mm to (166.0, 65.7), turned to 270 degrees
- moved J19 122.4 mm to (153.3, 65.7), turned to 270 degrees
- moved J18 108.6 mm to (147.0, 65.7), turned to 270 degrees
- moved J15 103.0 mm to (152.3, 55.0), turned to 90 degrees
- moved J14 91.2 mm to (145.9, 55.0), turned to 90 degrees
- moved C100 38.5 mm to (187.4, 14.4)
- moved J12 34.5 mm to (133.3, 55.0), turned to 90 degrees
- moved C70 6.30 mm to (160.7, 57.4)
- moved D10 6.30 mm to (160.9, 56.0)
- moved J16 6.30 mm to (158.6, 55.0)
- moved JP14 6.30 mm to (159.1, 50.9)
- moved JP17 6.30 mm to (158.6, 51.5)
- moved JP18 6.30 mm to (159.1, 58.5)
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Connections:
- D11 pad 1: /IO6/IO -> /IO8/IO
- D12 pad 1: /IO7/IO -> /IO9/IO
- D13 pad 1: /IO8/IO -> /IO10/IO
- D14 pad 1: /IO9/IO -> /IO12/IO
- D15 pad 1: /IO10/IO -> /IO11/IO
- R39 pad 1: /IO6/IO -> /IO8/IO
- R41 pad 1: /IO7/IO -> /IO9/IO
- R44 pad 1: /IO8/IO -> /IO10/IO
- R47 pad 1: /IO9/IO -> /IO12/IO
- R51 pad 1: /IO10/IO -> /IO11/IO
Routing:
- net /IO10/IO: track 8.43 -> 0.00 mm
- net /IO11/IO: track 0.00 -> 8.43 mm

Commit message: replicate
Parts:
- C64, C67, C68, C69, C71, C72, C73, C74, C76, C77, D11, D12, D13, D14, D16, D17, D6, D7, D8, D9, JP10, JP11, JP12, JP13, JP19, JP2, JP20, JP21, JP22, JP23, JP24, JP25, JP26, JP27, JP28, JP29, JP3, JP30, JP34, JP35, JP36, JP37, JP38, JP39, JP4, JP5, JP6, JP7, JP8, JP9, Q10, Q11, Q12, Q13, Q15, Q16, Q3, Q6, Q7, Q8, R30, R31, R32, R33, R34, R35, R39, R40, R41, R43, R44, R45, R47, R49, R53, R54, R55, R56, R6, R7: moved to B.Cu
- moved R40 174.5 mm to (138.3, 66.7), turned to 180 degrees
- moved JP20 171.8 mm to (140.7, 69.2), turned to 270 degrees
- moved Q10 170.9 mm to (138.7, 68.8)
- moved JP21 168.8 mm to (140.2, 62.2), turned to 270 degrees
- moved JP19 166.0 mm to (140.2, 69.8), turned to 180 degrees
- moved R39 162.1 mm to (141.6, 69.8), turned to 180 degrees
- moved D11 161.7 mm to (138.3, 64.7), turned to 180 degrees
- moved C71 158.0 mm to (138.6, 63.3), turned to 180 degrees
- moved JP5 149.1 mm to (140.1, 50.9)
- moved D7 148.4 mm to (142.0, 56.0)
- moved R49 147.7 mm to (163.6, 66.7), turned to 180 degrees
- moved JP7 147.2 mm to (140.2, 58.5), turned to 90 degrees
- moved Q6 145.1 mm to (141.6, 51.9), turned to 180 degrees
- moved JP29 145.0 mm to (166.0, 69.2), turned to 270 degrees
- moved Q13 144.3 mm to (164.0, 68.8)
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Routing:
- net +12V: track 49.5 -> 19.0 mm
- net +24V: track 117.5 -> 148.0 mm, vias 25 -> 30
- net /IO6/IO: track 0.00 -> 11.0 mm
- net /IO4/IO: track 0.00 -> 11.0 mm
- net /IO3/IO: track 0.00 -> 11.0 mm
- net /IO2/IO: track 0.00 -> 11.0 mm
- net /IO1/IO: track 0.00 -> 11.0 mm
- net /IO8/IO: track 0.00 -> 8.43 mm
- net /IO7/IO: track 0.00 -> 8.43 mm
- net /IO12/IO: track 0.00 -> 8.43 mm
- net /IO10/IO: track 0.00 -> 8.43 mm
- net /IO9/IO: track 0.00 -> 8.43 mm
- net Net-(JP37-Pad2): track 0.00 -> 3.74 mm
- net Net-(JP28-Pad2): track 0.00 -> 3.74 mm
- net Net-(JP25-Pad2): track 0.00 -> 3.74 mm
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- added copper zone on B.Cu, net Net-(C64-Pad1)
- added copper zone on B.Cu, net Net-(C67-Pad1)
- added copper zone on B.Cu, net Net-(C68-Pad1)
- added copper zone on B.Cu, net Net-(C69-Pad1)
- added copper zone on B.Cu, net Net-(C71-Pad1)
- added copper zone on B.Cu, net Net-(C72-Pad1)
- added copper zone on B.Cu, net Net-(C73-Pad1)
- added copper zone on B.Cu, net Net-(C74-Pad1)
- added copper zone on B.Cu, net Net-(C76-Pad1)
- added copper zone on B.Cu, net Net-(C77-Pad1)
- added copper zone on B.Cu, net Net-(J12-Pad3)
- added copper zone on B.Cu, net Net-(J13-Pad3)
- added copper zone on B.Cu, net Net-(J14-Pad3)
- added copper zone on B.Cu, net Net-(J15-Pad3)
- added copper zone on B.Cu, net Net-(J17-Pad3)
- added copper zone on B.Cu, net Net-(J18-Pad3)
- added copper zone on B.Cu, net Net-(J19-Pad3)
- added copper zone on B.Cu, net Net-(J20-Pad3)
- added copper zone on B.Cu, net Net-(J22-Pad3)
- added copper zone on B.Cu, net Net-(J23-Pad3)
- added copper zone on B.Cu, net Net-(JP11-Pad1)
- added copper zone on B.Cu, net Net-(JP11-Pad2)
- added copper zone on B.Cu, net Net-(JP19-Pad1)
- added copper zone on B.Cu, net Net-(JP19-Pad2)
- added copper zone on B.Cu, net Net-(JP2-Pad1)
- added copper zone on B.Cu, net Net-(JP2-Pad2)
- added copper zone on B.Cu, net Net-(JP22-Pad1)
- added copper zone on B.Cu, net Net-(JP22-Pad2)
- added copper zone on B.Cu, net Net-(JP25-Pad1)
- added copper zone on B.Cu, net Net-(JP25-Pad2)
- added copper zone on B.Cu, net Net-(JP28-Pad1)
- added copper zone on B.Cu, net Net-(JP28-Pad2)
- added copper zone on B.Cu, net Net-(JP34-Pad1)
- added copper zone on B.Cu, net Net-(JP34-Pad2)
- added copper zone on B.Cu, net Net-(JP37-Pad1)
- added copper zone on B.Cu, net Net-(JP37-Pad2)
- added copper zone on B.Cu, net Net-(JP5-Pad1)
- added copper zone on B.Cu, net Net-(JP5-Pad2)
- added copper zone on B.Cu, net Net-(JP8-Pad1)
- added copper zone on B.Cu, net Net-(JP8-Pad2)

Commit message: routing
Parts:
- removed C100, C111, C89: 100u, Capacitor_SMD:CP_Elec_6.3x7.7
- removed C54: 220u, Capacitor_SMD:CP_Elec_6.3x7.7
- removed C58, C66: 4.7u, _Generic:1210_CAP
- C53: value 100u -> 220u
- C55, C56, C57, C62, C63, C65, F2, F3: moved to B.Cu
- R4, R5: value 1k -> 10k
- moved C1 186.5 mm to (189.0, 182.4)
- moved C10 186.5 mm to (192.0, 182.4)
- moved C11 186.5 mm to (195.0, 182.6)
- moved C13 186.5 mm to (188.5, 187.0)
- moved C14 186.5 mm to (192.0, 184.3)
- moved C18 186.5 mm to (168.5, 172.7)
- moved C19 186.5 mm to (185.5, 188.9)
- moved C21 186.5 mm to (173.7, 168.7)
- moved C26 186.5 mm to (198.0, 180.7)
- moved C31 186.5 mm to (195.0, 184.5)
- moved C4 186.5 mm to (182.5, 187.0)
- moved C6 186.5 mm to (182.5, 188.9)
- moved C8 186.5 mm to (185.5, 187.0)
- moved C9 186.5 mm to (189.0, 184.3)
- moved D4 186.5 mm to (170.2, 170.8)
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Connections:
- D3 pad 1: Net-(D3-Pad1) -> GND
- D5 pad 1: Net-(D5-Pad1) -> GND
- J11 pad 1: Net-(D5-Pad1) -> Net-(C55-Pad1)
- J11 pad 2: Net-(C55-Pad1) -> Net-(J11-Pad2)
- J11 pad 3: Net-(D3-Pad1) -> Net-(C62-Pad1)
- J11 pad 4: Net-(C62-Pad1) -> Net-(J11-Pad4)
- Q4 pad 3: Net-(D3-Pad1) -> Net-(J11-Pad4)
- Q5 pad 3: Net-(D5-Pad1) -> Net-(J11-Pad2)
- R4 pad 1: +12V -> /Peripherals/POWER_OUT2
- R5 pad 1: +12V -> /Peripherals/POWER_OUT1
Routing:
- net GND: track 155.5 -> 267.6 mm
- net +24V: track 148.0 -> 124.8 mm, vias 30 -> 29
- net /IO6/IO: track 11.0 -> 25.8 mm
- net +12V: track 19.0 -> 33.2 mm, vias 1 -> 9
- net /IO2/IO: track 11.0 -> 24.2 mm
- net /IO4/IO: track 11.0 -> 24.1 mm
- net /IO5/IO: track 11.0 -> 24.1 mm
- net /IO3/IO: track 11.0 -> 24.1 mm
- net +5V: track 16.9 -> 24.8 mm, vias 6 -> 7
- net /IO1/IO: track 11.0 -> 17.4 mm
- net Net-(C37-Pad2): track 4.69 -> 0.00 mm
- net Net-(D1-Pad1): track 0.00 -> 4.41 mm
- net Net-(Q5-Pad2): track 0.00 -> 4.10 mm
- net Net-(R2-Pad2): track 0.00 -> 3.77 mm
- net Net-(R11-Pad1): track 0.00 -> 3.29 mm
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- added copper zone on B.Cu, net +12V
- added copper zone on B.Cu, net +5V
- added copper zone on F.Cu, net DCIN-
- added copper zone on F.Cu, net Net-(C28-Pad1)
- added copper zone on F.Cu, net Net-(C28-Pad2)
- added copper zone on F.Cu, net Net-(C29-Pad2)
- added copper zone on F.Cu, net Net-(C37-Pad1)
- added copper zone on F.Cu, net Net-(C37-Pad2)
- added copper zone on F.Cu, net Net-(C39-Pad2)
- added copper zone on B.Cu, net Net-(C55-Pad1)
- added copper zone on B.Cu, net Net-(C62-Pad1)
- added copper zone on B.Cu, net Net-(F1-Pad1)
- added copper zone on F.Cu, net Net-(F1-Pad1)
- added copper zone on F.Cu, net Net-(J11-Pad2)
- added copper zone on F.Cu, net Net-(J11-Pad4)
- added copper zone on F.Cu, net Net-(R11-Pad1)
- added copper zone on F.Cu, net Net-(R15-Pad1)
Other:
- board size 80 x 58.8 mm -> 75 x 55 mm
- board text removed: "Kajikia"
- board text removed: "P0.26"
