File: hardware/c3dpb.kicad_pcb (KiCad board)
At the start: 4 copper layers, 75 x 55 mm, 329 parts, among them IC1 TMC2209, IC2 TMC2209, IC3 TMC2209, IC4 TMC2209, J1 Conn_01x01, J10 Conn_01x04, J100 Conn_01x01, J101 Conn_01x01, J102 Conn_01x01, J11 Screw_Terminal_01x04, J12 Conn_01x03, J13 Conn_01x03, J14 Conn_01x03, J15 Conn_01x03, J16 Conn_01x03, J17 Conn_01x03, J18 Conn_01x03, J19 Conn_01x03, J2 Conn_01x01, J20 Conn_01x03, J21 Conn_01x03, J22 Conn_01x03, J23 Conn_01x03, J24 Conn_01x01, J3 Conn_01x01, J39 Screw_Terminal_01x02, J4 Conn_01x01, J44 Conn_01x01, J45 Conn_01x01, J48 Conn_01x01, J49 Conn_01x01, J5 Conn_01x01, J50 Conn_01x01, J51 Conn_01x01, J53 Conn_01x01, J54 Conn_01x01, J55 Conn_01x01, J56 Conn_01x01, J57 Conn_01x01, J58 Conn_01x01, J59 Conn_01x01, J6 Conn_01x01, J60 USB_C_Receptacle, J62 Conn_01x02, J68 Conn_01x01, J69 Conn_01x01, J7 Conn_01x04, J70 Conn_01x01, J71 Conn_01x02, J72 Conn_01x02, J73 Conn_01x02, J8 Conn_01x04, J9 Conn_01x04, J94 Conn_01x01, J95 Conn_01x01, J96 Conn_01x01, J98 Conn_01x01, J99 Conn_01x01, Q1 AON7418, Q10 AO3402, Q11 AO3402, Q12 AO3402, Q13 AO3402, Q14 AO3402, Q15 AO3402, Q16 AO3402, Q2 AO3400, Q3 AO3402, Q4 AON7418, Q5 AON7418, Q6 AO3402, Q7 AO3402, Q8 AO3402, Q9 AO3402, SW1 3x6mm, U1 ATSAMD51J19A-M, U2 LM1117-3.3, U3 SY8303, U4 SY8303, U5 MAX6675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

Commit message: pcb v1
Parts:
- removed C198: 10u, _Generic:0603_CAP
- removed J100, J101, J102, J44, J50, J51, J53, J54, J55, J68, J69, J70, J96, J98, J99: Conn_01x01, _Generic:PinHeader_2.54mm_1P
- removed JP1: SolderJumper_2_Open, _Generic:Solder Jumper 2P
- removed JP16: SolderJumper_3_Open, _Generic:Solder Jumper 3P
- removed SW1: 3x6mm, _Generic:Switch_3x4mm
- added C54: 100n, _Generic:0603_CAP, B.Cu at (120.6, 92.0)
- added C58: 100n, _Generic:0603_CAP, B.Cu at (133.6, 92.0)
- added C66: 100n, _Generic:0603_CAP, B.Cu at (146.6, 92.0)
- added C79: 100n, _Generic:0603_CAP, B.Cu at (159.6, 92.0)
- added C89: 4.7u, _Generic:1210_CAP, B.Cu at (171.5, 84.1)
- added FB2: 220r/100mhz, _Generic:0603_IND, B.Cu at (126.3, 77.2)
- added J25: Conn_01x01, _Generic:PinHeader_2.54mm_1P, F.Cu at (156.7, 82.9)
- added J26: Conn_01x01, _Generic:PinHeader_2.54mm_1P, F.Cu at (144.0, 82.9)
- added J27: Conn_01x01, _Generic:PinHeader_2.54mm_1P, F.Cu at (141.5, 80.4)
- added J28: Conn_01x01, _Generic:PinHeader_2.54mm_1P, F.Cu at (144.0, 80.4)
- added J29: Conn_01x01, _Generic:PinHeader_2.54mm_1P, F.Cu at (146.6, 80.4)
- added J30: Conn_01x01, _Generic:PinHeader_2.54mm_1P, F.Cu at (149.1, 80.4)
- added J31: Conn_01x01, _Generic:PinHeader_2.54mm_1P, F.Cu at (151.6, 82.9)
- added J32: Conn_01x01, _Generic:PinHeader_2.54mm_1P, F.Cu at (149.1, 82.9)
- added J33: Conn_01x01, _Generic:PinHeader_2.54mm_1P, F.Cu at (133.9, 80.4)
- added J34: Conn_01x01, _Generic:PinHeader_2.54mm_1P, F.Cu at (136.4, 80.4)
- C10, C11, C12, C19, C2, C21, C22, C4, C45, C48, C6, C7, C8, C9, JP15, L4, L5, R21, R22, R23: moved to B.Cu
- C13, C14: value 100n -> 10u; moved to B.Cu
- C26: value 10u -> 100n; moved to B.Cu
- C31: value 10u -> 4.7u; footprint _Generic:0603_CAP -> _Generic:1210_CAP; moved to B.Cu
- FB1: footprint _Generic:0805_IND -> _Generic:0603_IND; moved to B.Cu
- LS1, U5: moved to F.Cu
- U2: value LM1117-3.3 -> SE5218ALG-LF; footprint Package_TO_SOT_SMD:SOT-223-3_TabPin2 -> Package_TO_SOT_SMD:SOT-23-5
- moved C14 126.2 mm to (125.2, 77.2), turned to 270 degrees
- moved C19 125.3 mm to (128.7, 77.2), turned to 270 degrees
- moved C26 125.2 mm to (127.5, 77.2), turned to 270 degrees
- moved C8 123.8 mm to (122.0, 80.7)
- moved C4 123.3 mm to (122.0, 79.5)
- moved C2 122.1 mm to (130.8, 80.2), turned to 180 degrees
- moved C6 119.2 mm to (130.8, 81.4), turned to 180 degrees
- moved C10 118.9 mm to (122.3, 86.0), turned to 90 degrees
- moved C13 118.3 mm to (130.8, 83.7), turned to 180 degrees
- moved R42 116.6 mm to (151.6, 78.5), turned to 180 degrees
- moved C12 116.0 mm to (130.8, 82.5), turned to 180 degrees
- moved C11 115.9 mm to (130.8, 86.0), turned to 180 degrees
- moved C7 115.7 mm to (123.5, 86.0), turned to 90 degrees
- moved C9 115.2 mm to (130.8, 84.8), turned to 180 degrees
- moved C18 113.7 mm to (120.2, 69.8), turned to 180 degrees
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Connections:
- C12 pad 1: +3V3 -> /VDDCORE
- C13 pad 1: +3V3 -> /VDDCORE
- C19 pad 1: +3V3 -> /VDDANA
- C26 pad 1: +3V3 -> /VDDANA
- C31 pad 1: +3V3 -> Net-(C31-Pad1)
- C59 pad 1: /P0.25_TH2 -> /TH3
- C60 pad 1: /P0.24_TH1 -> /TH1
- C61 pad 1: /P0.23_TH0 -> /TH2
- D10 pad 1: /IO5/IO -> /IO5
- D11 pad 1: /IO8/IO -> /IO8
- D12 pad 1: /IO9/IO -> /IO9
- D13 pad 1: /IO10/IO -> /IO10
- D14 pad 1: /IO12/IO -> /IO12
- D15 pad 1: /IO11/IO -> /IO11
- D16 pad 1: /IO6/IO -> /IO6
- D17 pad 1: /IO7/IO -> /IO7
- D6 pad 1: /IO1/IO -> /IO1
- D7 pad 1: /IO2/IO -> /IO2
- D8 pad 1: /IO3/IO -> /IO3
- D9 pad 1: /IO4/IO -> /IO4
- H1 pad 1: GND -> Net-(H1-Pad1)
- IC1 pad 10: /Driver 2/AD1 -> GND
- IC1 pad 11: /DRV2_DIAG -> /DRV1_DIAG
- IC1 pad 14: /DRV_UART -> /DRV1_UART
- IC1 pad 15: Net-(IC1-Pad15) -> +3V3
- IC1 pad 16: /DRV2_STEP -> /DRV1_STEP
- IC1 pad 19: /DRV2_DIR -> /DRV1_DIR
- IC1 pad 2: /DRV2_EN -> GND
- IC1 pad 20: Net-(IC1-Pad20) -> GND
- IC1 pad 7: Net-(IC1-Pad7) -> GND
- IC1 pad 9: +3V3 -> GND
- IC2 pad 10: +3V3 -> GND
- IC2 pad 11: /DRV3_DIAG -> /DRV2_DIAG
- IC2 pad 14: /DRV_UART -> /DRV2_UART
- IC2 pad 15: Net-(IC2-Pad15) -> +3V3
- IC2 pad 16: /DRV3_STEP -> /DRV2_STEP
- IC2 pad 19: /DRV3_DIR -> /DRV2_DIR
- IC2 pad 2: /DRV3_EN -> GND
- IC2 pad 20: Net-(IC2-Pad20) -> GND
- IC2 pad 7: Net-(IC2-Pad7) -> GND
- IC2 pad 9: /Driver 3/AD0 -> GND
- IC3 pad 10: +3V3 -> GND
- IC3 pad 11: /DRV4_DIAG -> /DRV3_DIAG
- IC3 pad 14: /DRV_UART -> /DRV3_UART
- IC3 pad 15: Net-(IC3-Pad15) -> +3V3
- IC3 pad 16: /DRV4_STEP -> /DRV3_STEP
- IC3 pad 19: /DRV4_DIR -> /DRV3_DIR
- IC3 pad 2: /DRV4_EN -> GND
- IC3 pad 20: Net-(IC3-Pad20) -> GND
- IC3 pad 7: Net-(IC3-Pad7) -> GND
- IC3 pad 9: +3V3 -> GND
- IC4 pad 10: /Driver 1/AD1 -> GND
- IC4 pad 11: /DRV1_DIAG -> /DRV4_DIAG
- IC4 pad 14: /DRV_UART -> /DRV4_UART
- IC4 pad 15: Net-(IC4-Pad15) -> +3V3
- IC4 pad 16: /DRV1_STEP -> /DRV4_STEP
- IC4 pad 19: /DRV1_DIR -> /DRV4_DIR
- IC4 pad 2: /DRV1_EN -> GND
- IC4 pad 20: Net-(IC4-Pad20) -> GND
- IC4 pad 7: Net-(IC4-Pad7) -> GND
- IC4 pad 9: /Driver 1/AD0 -> GND
- J2 pad 1: /BUZZER -> /SWDIO
- J3 pad 1: Net-(J3-Pad1) -> /I2C_SDA
- J4 pad 1: Net-(J4-Pad1) -> /I2C_SCL
- J6 pad 1: Net-(J6-Pad1) -> /BUZZER
- J60 pad A4: Net-(C198-Pad1) -> Net-(C31-Pad1)
- J60 pad A9: Net-(C198-Pad1) -> Net-(C31-Pad1)
- J60 pad B4: Net-(C198-Pad1) -> Net-(C31-Pad1)
- J60 pad B9: Net-(C198-Pad1) -> Net-(C31-Pad1)
- J71 pad 1: /P0.23_TH0 -> /TH2
- J72 pad 1: /P0.24_TH1 -> /TH1
- J73 pad 1: /P0.25_TH2 -> /TH3
- JP15 pad 1: Net-(C198-Pad1) -> Net-(C31-Pad1)
- R16 pad 2: Net-(JP1-Pad2) -> /BUZZER
- R30 pad 1: /IO2/IO -> /IO2
- R32 pad 1: /IO3/IO -> /IO3
- R34 pad 1: /IO4/IO -> /IO4
- R36 pad 1: /IO5/IO -> /IO5
- R37 pad 1: Net-(JP16-Pad2) -> +3V3
- R37 pad 2: /SCL -> /I2C_SCL
- R39 pad 1: /IO8/IO -> /IO8
- R4 pad 1: /Peripherals/POWER_OUT2 -> /POW2
- R41 pad 1: /IO9/IO -> /IO9
- R42 pad 1: Net-(JP16-Pad2) -> +3V3
- R42 pad 2: /SDA -> /I2C_SDA
- R44 pad 1: /IO10/IO -> /IO10
- R46 pad 2: /P0.25_TH2 -> /TH3
- R47 pad 1: /IO12/IO -> /IO12
- R48 pad 2: /P0.24_TH1 -> /TH1
- R5 pad 1: /Peripherals/POWER_OUT1 -> /POW1
- R50 pad 2: /P0.23_TH0 -> /TH2
- R51 pad 1: /IO11/IO -> /IO11
- R53 pad 1: /IO6/IO -> /IO6
- R55 pad 1: /IO7/IO -> /IO7
- R6 pad 1: /IO1/IO -> /IO1
- U1 pad 1: Net-(J3-Pad1) -> /I2C_SDA
- U1 pad 10: Net-(U1-Pad10) -> /IO12
- U1 pad 11: Net-(U1-Pad11) -> /IO5
- U1 pad 12: Net-(U1-Pad12) -> /IO11
- U1 pad 13: /P1.18_ADV -> /IO4
- U1 pad 14: /P1.19_ADV -> /IO10
- U1 pad 15: /P1.22_ADV -> /IO3
- U1 pad 16: /P1.25_ADV -> /IO9
- U1 pad 17: /P1.26_ADV -> /IO2
- U1 pad 18: /P1.28_ADV -> /IO8
- U1 pad 19: /P1.29_ADV -> /IO1
- U1 pad 2: Net-(J4-Pad1) -> /I2C_SCL
- U1 pad 20: /P0.22_ADV -> /IO7
- U1 pad 21: /VDDIO -> +3V3
- U1 pad 22: Net-(U1-Pad22) -> GND
- U1 pad 23: /DRV3_STEP -> /DRV1_DIR
- U1 pad 24: /DRV4_STEP -> /DRV1_STEP
- U1 pad 25: /DRV2_DIR -> /DRV1_UART
- U1 pad 26: /DRV2_EN -> /DRV1_DIAG
- U1 pad 27: /DRV3_DIR -> /DRV2_DIR
- U1 pad 28: /DRV3_EN -> /DRV2_STEP
- U1 pad 29: /DRV1_DIAG -> /POW2
- U1 pad 30: /DRV2_DIAG -> /POW1
- U1 pad 31: /DRV1_STEP -> /DRV2_UART
- U1 pad 32: /DRV2_STEP -> /DRV2_DIAG
- U1 pad 33: Net-(U1-Pad22) -> GND
- U1 pad 34: /VDDIO -> +3V3
- U1 pad 35: /DRV_UART -> /BUZZER
- U1 pad 36: /DRV_UART -> Net-(J25-Pad1)
- U1 pad 37: /P2.3_POW -> /DRV3_DIR
- U1 pad 38: /P2.4_POW -> /DRV3_STEP
- U1 pad 39: /DRV4_DIR -> /DRV3_UART
- U1 pad 4: Net-(J6-Pad1) -> /TH3
- U1 pad 40: /DRV4_EN -> /DRV3_DIAG
- U1 pad 41: /DRV3_DIAG -> /DRV4_DIR
- U1 pad 42: /DRV4_DIAG -> /DRV4_STEP
- U1 pad 43: /DRV1_DIR -> /DRV4_UART
- U1 pad 44: /DRV1_EN -> /DRV4_DIAG
- U1 pad 47: Net-(U1-Pad22) -> GND
- U1 pad 48: /VDDIO -> +3V3
- U1 pad 5: Net-(U1-Pad5) -> /TH2
- U1 pad 54: Net-(U1-Pad22) -> GND
- U1 pad 56: /VDDIO -> +3V3
- U1 pad 58: /BUZZER -> /SWDIO
- U1 pad 6: Net-(U1-Pad6) -> /TH1
- U1 pad 61: Net-(U1-Pad61) -> /SPI_CS
- U1 pad 62: Net-(U1-Pad62) -> /SPI_MISO
- U1 pad 63: Net-(U1-Pad63) -> /SPI_MOSI
- U1 pad 64: Net-(U1-Pad64) -> /SPI_SCK
- U1 pad 65: Net-(U1-Pad22) -> GND
- U1 pad 7: Net-(U1-Pad22) -> GND
- U1 pad 9: Net-(U1-Pad9) -> /IO6
- U2 pad 1: GND -> Net-(C20-Pad1)
- U2 pad 2: +3V3 -> GND
- U5 pad 5: /DRV_SCK -> /SPI_SCK
- U5 pad 6: /MAX1_CS -> /SPI_CS
- U5 pad 7: /DRV_MISO -> /SPI_MISO
- U6 pad 2: /Peripherals/POWER_OUT1 -> /POW1
- U6 pad 4: /Peripherals/POWER_OUT2 -> /POW2
Routing:
- net +3V3: track 0.50 -> 210.7 mm, vias 0 -> 23
- net GND: track 267.6 -> 471.5 mm, vias 120 -> 363
- net /IO6: track 0.00 -> 68.4 mm, vias 0 -> 1
- net /TH1: track 0.00 -> 64.8 mm
- net /IO5: track 0.00 -> 63.2 mm, vias 0 -> 1
- net /IO4: track 0.00 -> 57.8 mm, vias 0 -> 1
- net /TH2: track 0.00 -> 55.9 mm
- net /IO12: track 0.00 -> 53.7 mm, vias 0 -> 1
- net /IO3: track 0.00 -> 52.6 mm, vias 0 -> 1
- net /TH3: track 0.00 -> 48.7 mm
- net /IO2: track 0.00 -> 48.5 mm, vias 0 -> 1
- net /IO11: track 0.00 -> 48.4 mm, vias 0 -> 1
- net +5V: track 24.8 -> 73.1 mm, vias 7 -> 18
- net /BUZZER: track 0.00 -> 46.0 mm, vias 0 -> 4
- net /IO1: track 0.00 -> 44.1 mm, vias 0 -> 1
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- added copper zone on B.Cu, net +3V3
- added copper zone on F.Cu, net +3V3
- added copper zone on B.Cu, net Net-(C31-Pad1)
- added copper zone on F.Cu, net Net-(C31-Pad1)
- added copper zone on B.Cu, net Net-(FB1-Pad2)
Other:
- copper layers 4 -> 2
- rule solder_mask_min_width: 0.25 -> 0.15
- board text added: "12"
- board text added: "24"
- board text added: "24v"
- board text added: "3.3V"
- board text added: "5"
- board text added: "A1"
- board text added: "A2"
- board text added: "B1"
- board text added: "B2"
- board text added: "BUZ"
- board text added: "CLK"
- board text added: "DI"
- board text added: "DIO"
- board text added: "DO"
- board text added: "DRV1"
- board text added: "DRV2"
- board text added: "DRV3"
- board text added: "DRV4"
- board text added: "GND"
- board text added: "JLCJLCJLCJLC"
- board text added: "PA0"
- board text added: "PA03"
- board text added: "PA04"
- board text added: "PA05"
- board text added: "PA06"
- board text added: "PA07"
- board text added: "PA08"
- board text added: "PA09"
- board text added: "PA1"
- board text added: "PA10"
- board text added: "PA11"
- board text added: "PA12"
- board text added: "PA13"
- board text added: "PA16"
- board text added: "PA17"
- board text added: "PA2"
- board text added: "PA27"
- board text added: "PA30"
- board text added: "PA31"
- board text added: "PB0"
- board text added: "PB04"
- board text added: "PB05"
- board text added: "PB06"
- board text added: "PB07"
- board text added: "PB08"
- board text added: "PB09"
- board text added: "PB1"
- board text added: "PB2"
- board text added: "PB22"
- board text added: "PB23"
- board text added: "PB3"
- board text added: "PB30"
- board text added: "PB31"
- board text added: "PWR"
- board text added: "RST"
- board text added: "SCK"
- board text added: "SCL"
- board text added: "SDA"
- board text removed: "24V"
- board text removed: "P0.23"
- board text removed: "P0.24"
- board text removed: "P0.25"

Commit message: pcb version 1.1
Parts:
- removed C29, C39: 47p, _Generic:0603_CAP
- removed L1: 1u, _Generic:0805_IND
- added D18: MSK4010, _Generic:SOD-523_DIODE, B.Cu at (108.2, 77.5)
- added D19: MSK4010, _Generic:SOD-523_DIODE, B.Cu at (108.2, 64.8)
- C107, C49, C85, C96: value 2.2u -> 10u
- C31, C89: value 4.7u -> 22u
- C64, C67, C68, C69, C70, C71, C72, C73, C74, C75, C76, C77: value 4.7u -> 1u; footprint _Generic:0805_CAP -> _Generic:0603_CAP
- D1: moved to B.Cu
- FB1: value Ferrite_Bead_Small -> 470r/100mhz
- FB2: value 220r/100mhz -> 470r/100mhz
- FB3: renamed from L4; value 470 -> 470r/100mhz
- FB4: renamed from L5; value 470 -> 470r/100mhz
- Q2: value AO3400 -> AO3402
- U3, U4: footprint Package_TO_SOT_SMD:TSOT-23-8 -> _Generic:TSOT-23-8
- moved C18 2.88 mm to (123.0, 69.9)
- moved R9 1.02 mm to (114.8, 95.9)
- moved R14 0.96 mm to (129.3, 71.3), turned to 0 degrees
- moved D4 0.94 mm to (129.3, 69.9), turned to 180 degrees
- moved R12 0.90 mm to (120.5, 55.4), turned to 0 degrees
- moved R17 0.90 mm to (129.2, 55.4), turned to 0 degrees
- moved C20 0.80 mm to (123.0, 71.3), turned to 0 degrees
- moved R8 0.78 mm to (114.8, 97.3)
- moved R13 0.65 mm to (120.5, 54.0)
- moved R18 0.65 mm to (129.2, 54.0)
- moved C14 0.50 mm to (124.7, 77.2)
- moved R4 0.40 mm to (121.1, 71.8)
- moved R11 0.40 mm to (120.5, 52.5)
- moved C9 0.35 mm to (130.8, 85.2)
- moved C11 0.35 mm to (130.8, 86.3)
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Connections:
- C20 pad 1: Net-(C20-Pad1) -> +5V
- U2 pad 1: Net-(C20-Pad1) -> +5V
- U2 pad 3: Net-(C20-Pad1) -> +5V
Routing:
- net Net-(C20-Pad1): track 9.29 -> 0.00 mm
- net /VDDANA: track 9.03 -> 14.9 mm
- net Net-(R15-Pad1): track 0.00 -> 4.01 mm
- net Net-(R12-Pad2): track 0.00 -> 3.43 mm
- net GND: track 471.5 -> 468.7 mm, vias 363 -> 358
- net +5V: track 73.1 -> 71.0 mm
- net /VDDCORE: track 3.47 -> 4.62 mm
- net Net-(C48-Pad1): track 10.2 -> 9.12 mm
- net Net-(R17-Pad2): track 4.19 -> 3.43 mm
- net +3V3: track 210.7 -> 211.4 mm
- net Net-(D1-Pad1): track 4.41 -> 4.04 mm, vias 0 -> 1
- removed copper zone on F.Cu, net Net-(R11-Pad1)
- removed copper zone on F.Cu, net Net-(R12-Pad2)
- removed copper zone on F.Cu, net Net-(R15-Pad1)
- removed copper zone on F.Cu, net Net-(R17-Pad2)
Other:
- board text added: "C3DPB v1.1"
