File: hardware/io.sch (KiCad schematic (older format))
At the start: 9 parts, among them J12 Conn_01x03, Q3 AO3402

Commit message: new con
Changed lines of the file:
@@
 $Descr A4 11693 8268
 encoding utf-8
-Sheet 12 17
+Sheet 8 19
 Title ""
 Date ""
@@
 AR Path="/5DC02A6B/5DCA99CE" Ref="J16"  Part="1"
 AR Path="/5DC28D35/5DCA99CE" Ref="J?"  Part="1"
-F 0 "J16" H 6730 3792 50  0000 L CNN
+AR Path="/5D38DAD4/5DCA99CE" Ref="J22"  Part="1"
+F 0 "J12" H 6730 3792 50  0000 L CNN
 F 1 "Conn_01x03" H 6730 3701 50  0001 L CNN
 F 2 "_Generic:JST_XH_3P" H 6650 3750 50  0001 C CNN
@@
 AR Path="/5DC02A6B/5DCA99CF" Ref="JP18"  Part="1"
 AR Path="/5DC28D35/5DCA99CF" Ref="JP?"  Part="1"
-F 0 "JP18" H 6558 3300 50  0000 L CNN
+AR Path="/5D38DAD4/5DCA99CF" Ref="JP36"  Part="1"
+F 0 "JP4" H 6558 3300 50  0000 L CNN
 F 1 "SolderJumper_4_Open" H 6400 3300 50  0001 C CNN
 F 2 "_Generic:SolderJumper_JST" H 6400 3300 50  0001 C CNN
@@
 AR Path="/5DC02A6B/5DB5A83A" Ref="#PWR0168"  Part="1"
 AR Path="/5DC28D35/5DB5A83A" Ref="#PWR?"  Part="1"
-F 0 "#PWR0168" H 6400 2950 50  0001 C CNN
+AR Path="/5D38DAD4/5DB5A83A" Ref="#PWR0198"  Part="1"
+F 0 "#PWR0112" H 6400 2950 50  0001 C CNN
 F 1 "+12V" H 6415 3273 50  0000 C CNN
 F 2 "" H 6400 3100 50  0001 C CNN
@@
 AR Path="/5DC02A6B/5DB5A841" Ref="#PWR0169"  Part="1"
 AR Path="/5DC28D35/5DB5A841" Ref="#PWR?"  Part="1"
-F 0 "#PWR0169" H 6150 2950 50  0001 C CNN
+AR Path="/5D38DAD4/5DB5A841" Ref="#PWR0199"  Part="1"
+F 0 "#PWR0113" H 6150 2950 50  0001 C CNN
 F 1 "+5V" H 6165 3273 50  0000 C CNN
 F 2 "" H 6150 3100 50  0001 C CNN
@@
 AR Path="/5DC02A6B/5DB5A848" Ref="JP14"  Part="1"
 AR Path="/5DC28D35/5DB5A848" Ref="JP?"  Part="1"
-F 0 "JP14" V 5450 3368 50  0000 L CNN
+AR Path="/5D38DAD4/5DB5A848" Ref="JP34"  Part="1"
+F 0 "JP2" V 5450 3368 50  0000 L CNN
 F 1 "SolderJumper_2_Open" H 5450 3300 50  0001 C CNN
 F 2 "_Generic:Solder Jumper 2P" H 5450 3300 50  0001 C CNN
@@
 AR Path="/5DC02A6B/5DB5A84E" Ref="JP17"  Part="1"
 AR Path="/5DC28D35/5DB5A84E" Ref="JP?"  Part="1"
-F 0 "JP17" V 5800 3232 50  0000 R CNN
+AR Path="/5D38DAD4/5DB5A84E" Ref="JP35"  Part="1"
+F 0 "JP3" V 5800 3232 50  0000 R CNN
 F 1 "SolderJumper_2_Open" H 5800 3300 50  0001 C CNN
 F 2 "_Generic:Solder Jumper 2P" H 5800 3300 50  0001 C CNN
@@
 AR Path="/5DC02A6B/5DB5A864" Ref="D10"  Part="1"
 AR Path="/5DC28D35/5DB5A864" Ref="D?"  Part="1"
-F 0 "D10" V 4554 3729 50  0000 L CNN
+AR Path="/5D38DAD4/5DB5A864" Ref="D16"  Part="1"
+F 0 "D6" V 4554 3729 50  0000 L CNN
 F 1 "3.6v" V 4645 3729 50  0000 L CNN
 F 2 "_Generic:SOD-523_DIODE" H 4600 3650 50  0001 C CNN
@@
 AR Path="/5DC02A6B/5DCA99D5" Ref="Q9"  Part="1"
 AR Path="/5DC28D35/5DCA99D5" Ref="Q?"  Part="1"
-F 0 "Q9" V 5700 3750 50  0000 C CNN
+AR Path="/5D38DAD4/5DCA99D5" Ref="Q15"  Part="1"
+F 0 "Q3" V 5700 3750 50  0000 C CNN
 F 1 "AO3402" V 5791 3750 50  0000 C CNN
 F 2 "_Generic:SOT-23" H 5650 3850 50  0001 C CNN
@@
 AR Path="/5DC02A6B/5DB5A87E" Ref="#PWR0170"  Part="1"
 AR Path="/5DC28D35/5DB5A87E" Ref="#PWR?"  Part="1"
-F 0 "#PWR0170" H 6100 3650 50  0001 C CNN
+AR Path="/5D38DAD4/5DB5A87E" Ref="#PWR0200"  Part="1"
+F 0 "#PWR0114" H 6100 3650 50  0001 C CNN
 F 1 "GND" H 6100 3750 50  0001 C CNN
 F 2 "" H 6100 3900 50  0001 C CNN
@@
 AR Path="/5DC02A6B/5DB5A885" Ref="#PWR0171"  Part="1"
 AR Path="/5DC28D35/5DB5A885" Ref="#PWR?"  Part="1"
-F 0 "#PWR0171" H 6650 2950 50  0001 C CNN
+AR Path="/5D38DAD4/5DB5A885" Ref="#PWR0202"  Part="1"
+F 0 "#PWR0115" H 6650 2950 50  0001 C CNN
 F 1 "+24V" H 6665 3273 50  0000 C CNN
 F 2 "" H 6650 3100 50  0001 C CNN
@@
 AR Path="/5DC02A6B/5DCA99D8" Ref="#PWR0172"  Part="1"
 AR Path="/5DC28D35/5DCA99D8" Ref="#PWR?"  Part="1"
-F 0 "#PWR0172" H 5000 3650 50  0001 C CNN
+AR Path="/5D38DAD4/5DCA99D8" Ref="#PWR0203"  Part="1"
+F 0 "#PWR0116" H 5000 3650 50  0001 C CNN
 F 1 "GND" H 5000 3750 50  0001 C CNN
 F 2 "" H 5000 3900 50  0001 C CNN
@@
 AR Path="/5DC02A6B/5DB5A893" Ref="C70"  Part="1"
 AR Path="/5DC28D35/5DB5A893" Ref="C?"  Part="1"
-F 0 "C70" H 6192 3646 50  0000 L CNN
+AR Path="/5D38DAD4/5DB5A893" Ref="C76"  Part="1"
+F 0 "C64" H 6192 3646 50  0000 L CNN
 F 1 "4.7u" H 6192 3555 50  0000 L CNN
 F 2 "_Generic:0805_CAP" H 6100 3600 50  0001 C CNN
@@
 AR Path="/5DC02A6B/5DB5A89A" Ref="R38"  Part="1"
 AR Path="/5DC28D35/5DB5A89A" Ref="R?"  Part="1"
-F 0 "R38" H 4930 3696 50  0000 R CNN
+AR Path="/5D38DAD4/5DB5A89A" Ref="R54"  Part="1"
+F 0 "R7" H 4930 3696 50  0000 R CNN
 F 1 "1meg" H 4930 3605 50  0000 R CNN
 F 2 "_Generic:0603_RES" V 4930 3650 50  0001 C CNN
@@
 AR Path="/5DC02A6B/5DCA99DB" Ref="R36"  Part="1"
 AR Path="/5DC28D35/5DCA99DB" Ref="R?"  Part="1"
-F 0 "R36" V 5207 3150 50  0000 C CNN
+AR Path="/5D38DAD4/5DCA99DB" Ref="R53"  Part="1"
+F 0 "R6" V 5207 3150 50  0000 C CNN
 F 1 "4.7k" V 5116 3150 50  0000 C CNN
 F 2 "_Generic:0603_RES" V 4930 3150 50  0001 C CNN

Commit message: pcb v1
Changed lines of the file:
@@
 $Descr A4 11693 8268
 encoding utf-8
-Sheet 8 19
+Sheet 10 19
 Title ""
 Date ""
@@
 AR Path="/5DC28D35/5DCA99CE" Ref="J?"  Part="1"
 AR Path="/5D38DAD4/5DCA99CE" Ref="J22"  Part="1"
-F 0 "J12" H 6730 3792 50  0000 L CNN
+F 0 "J22" H 6730 3792 50  0000 L CNN
 F 1 "Conn_01x03" H 6730 3701 50  0001 L CNN
 F 2 "_Generic:JST_XH_3P" H 6650 3750 50  0001 C CNN
@@
 AR Path="/5DC28D35/5DCA99CF" Ref="JP?"  Part="1"
 AR Path="/5D38DAD4/5DCA99CF" Ref="JP36"  Part="1"
-F 0 "JP4" H 6558 3300 50  0000 L CNN
+F 0 "JP36" H 6558 3300 50  0000 L CNN
 F 1 "SolderJumper_4_Open" H 6400 3300 50  0001 C CNN
 F 2 "_Generic:SolderJumper_JST" H 6400 3300 50  0001 C CNN
@@
 AR Path="/5DC28D35/5DB5A83A" Ref="#PWR?"  Part="1"
 AR Path="/5D38DAD4/5DB5A83A" Ref="#PWR0198"  Part="1"
-F 0 "#PWR0198" H 6400 2950 50  0001 C CNN
+F 0 "#PWR0122" H 6400 2950 50  0001 C CNN
 F 1 "+12V" H 6415 3273 50  0000 C CNN
 F 2 "" H 6400 3100 50  0001 C CNN
@@
 AR Path="/5DC28D35/5DB5A841" Ref="#PWR?"  Part="1"
 AR Path="/5D38DAD4/5DB5A841" Ref="#PWR0199"  Part="1"
-F 0 "#PWR0199" H 6150 2950 50  0001 C CNN
+F 0 "#PWR0124" H 6150 2950 50  0001 C CNN
 F 1 "+5V" H 6165 3273 50  0000 C CNN
 F 2 "" H 6150 3100 50  0001 C CNN
@@
 AR Path="/5DC28D35/5DB5A848" Ref="JP?"  Part="1"
 AR Path="/5D38DAD4/5DB5A848" Ref="JP34"  Part="1"
-F 0 "JP2" V 5450 3368 50  0000 L CNN
+F 0 "JP34" V 5450 3368 50  0000 L CNN
 F 1 "SolderJumper_2_Open" H 5450 3300 50  0001 C CNN
 F 2 "_Generic:Solder Jumper 2P" H 5450 3300 50  0001 C CNN
@@
 AR Path="/5DC28D35/5DB5A84E" Ref="JP?"  Part="1"
 AR Path="/5D38DAD4/5DB5A84E" Ref="JP35"  Part="1"
-F 0 "JP3" V 5800 3232 50  0000 R CNN
+F 0 "JP35" V 5800 3232 50  0000 R CNN
 F 1 "SolderJumper_2_Open" H 5800 3300 50  0001 C CNN
 F 2 "_Generic:Solder Jumper 2P" H 5800 3300 50  0001 C CNN
@@
 AR Path="/5DC28D35/5DB5A864" Ref="D?"  Part="1"
 AR Path="/5D38DAD4/5DB5A864" Ref="D16"  Part="1"
-F 0 "D6" V 4554 3729 50  0000 L CNN
+F 0 "D16" V 4554 3729 50  0000 L CNN
 F 1 "3.6v" V 4645 3729 50  0000 L CNN
 F 2 "_Generic:SOD-523_DIODE" H 4600 3650 50  0001 C CNN
@@
 AR Path="/5DC28D35/5DCA99D5" Ref="Q?"  Part="1"
 AR Path="/5D38DAD4/5DCA99D5" Ref="Q15"  Part="1"
-F 0 "Q3" V 5700 3750 50  0000 C CNN
+F 0 "Q15" V 5700 3750 50  0000 C CNN
 F 1 "AO3402" V 5791 3750 50  0000 C CNN
 F 2 "_Generic:SOT-23" H 5650 3850 50  0001 C CNN
@@
 AR Path="/5DC28D35/5DB5A87E" Ref="#PWR?"  Part="1"
 AR Path="/5D38DAD4/5DB5A87E" Ref="#PWR0200"  Part="1"
-F 0 "#PWR0200" H 6100 3650 50  0001 C CNN
+F 0 "#PWR0160" H 6100 3650 50  0001 C CNN
 F 1 "GND" H 6100 3750 50  0001 C CNN
 F 2 "" H 6100 3900 50  0001 C CNN
@@
 AR Path="/5DC28D35/5DB5A885" Ref="#PWR?"  Part="1"
 AR Path="/5D38DAD4/5DB5A885" Ref="#PWR0202"  Part="1"
-F 0 "#PWR0202" H 6650 2950 50  0001 C CNN
+F 0 "#PWR0161" H 6650 2950 50  0001 C CNN
 F 1 "+24V" H 6665 3273 50  0000 C CNN
 F 2 "" H 6650 3100 50  0001 C CNN
@@
 AR Path="/5DC28D35/5DCA99D8" Ref="#PWR?"  Part="1"
 AR Path="/5D38DAD4/5DCA99D8" Ref="#PWR0203"  Part="1"
-F 0 "#PWR0203" H 5000 3650 50  0001 C CNN
+F 0 "#PWR0162" H 5000 3650 50  0001 C CNN
 F 1 "GND" H 5000 3750 50  0001 C CNN
 F 2 "" H 5000 3900 50  0001 C CNN
@@
 AR Path="/5DC28D35/5DB5A893" Ref="C?"  Part="1"
 AR Path="/5D38DAD4/5DB5A893" Ref="C76"  Part="1"
-F 0 "C64" H 6192 3646 50  0000 L CNN
+F 0 "C76" H 6192 3646 50  0000 L CNN
 F 1 "4.7u" H 6192 3555 50  0000 L CNN
 F 2 "_Generic:0805_CAP" H 6100 3600 50  0001 C CNN
@@
 AR Path="/5DC28D35/5DB5A89A" Ref="R?"  Part="1"
 AR Path="/5D38DAD4/5DB5A89A" Ref="R54"  Part="1"
-F 0 "R7" H 4930 3696 50  0000 R CNN
+F 0 "R54" H 4930 3696 50  0000 R CNN
 F 1 "1meg" H 4930 3605 50  0000 R CNN
 F 2 "_Generic:0603_RES" V 4930 3650 50  0001 C CNN
@@
 AR Path="/5DC28D35/5DCA99DB" Ref="R?"  Part="1"
 AR Path="/5D38DAD4/5DCA99DB" Ref="R53"  Part="1"
-F 0 "R6" V 5207 3150 50  0000 C CNN
+F 0 "R53" V 5207 3150 50  0000 C CNN
 F 1 "4.7k" V 5116 3150 50  0000 C CNN
 F 2 "_Generic:0603_RES" V 4930 3150 50  0001 C CNN
