File: hardware/io_rev.sch (KiCad schematic (older format))
At the start: 9 parts, among them J17 Conn_01x03, Q10 AO3402

Commit message: routing
Changed lines of the file:
@@
 $Descr A4 11693 8268
 encoding utf-8
-Sheet 17 19
+Sheet 19 19
 Title ""
 Date ""
@@
 AR Path="/5DC58965/5DB5A825" Ref="J21"  Part="1"
 AR Path="/5D399F3E/5DB5A825" Ref="J23"  Part="1"
-F 0 "J21" H 6730 3792 50  0000 L CNN
+F 0 "J23" H 6730 3792 50  0000 L CNN
 F 1 "Conn_01x03" H 6730 3701 50  0001 L CNN
 F 2 "_Generic:JST_XH_3P" H 6650 3750 50  0001 C CNN
@@
 AR Path="/5DC58965/5DB5A832" Ref="JP33"  Part="1"
 AR Path="/5D399F3E/5DB5A832" Ref="JP39"  Part="1"
-F 0 "JP33" H 6558 3300 50  0000 L CNN
+F 0 "JP39" H 6558 3300 50  0000 L CNN
 F 1 "SolderJumper_4_Open" H 6400 3300 50  0001 C CNN
 F 2 "_Generic:SolderJumper_JST" H 6400 3300 50  0001 C CNN
@@
 AR Path="/5DC58965/5DCA99D0" Ref="#PWR0193"  Part="1"
 AR Path="/5D399F3E/5DCA99D0" Ref="#PWR0204"  Part="1"
-F 0 "#PWR0193" H 6400 2950 50  0001 C CNN
+F 0 "#PWR0204" H 6400 2950 50  0001 C CNN
 F 1 "+12V" H 6415 3273 50  0000 C CNN
 F 2 "" H 6400 3100 50  0001 C CNN
@@
 AR Path="/5DC58965/5DCA99D1" Ref="#PWR0194"  Part="1"
 AR Path="/5D399F3E/5DCA99D1" Ref="#PWR0205"  Part="1"
-F 0 "#PWR0194" H 6150 2950 50  0001 C CNN
+F 0 "#PWR0205" H 6150 2950 50  0001 C CNN
 F 1 "+5V" H 6165 3273 50  0000 C CNN
 F 2 "" H 6150 3100 50  0001 C CNN
@@
 AR Path="/5DC58965/5DCA99D2" Ref="JP31"  Part="1"
 AR Path="/5D399F3E/5DCA99D2" Ref="JP37"  Part="1"
-F 0 "JP31" V 5450 3368 50  0000 L CNN
+F 0 "JP37" V 5450 3368 50  0000 L CNN
 F 1 "SolderJumper_2_Open" H 5450 3300 50  0001 C CNN
 F 2 "_Generic:Solder Jumper 2P" H 5450 3300 50  0001 C CNN
@@
 AR Path="/5DC58965/5DCA99D3" Ref="JP32"  Part="1"
 AR Path="/5D399F3E/5DCA99D3" Ref="JP38"  Part="1"
-F 0 "JP32" V 5800 3232 50  0000 R CNN
+F 0 "JP38" V 5800 3232 50  0000 R CNN
 F 1 "SolderJumper_2_Open" H 5800 3300 50  0001 C CNN
 F 2 "_Generic:Solder Jumper 2P" H 5800 3300 50  0001 C CNN
@@
 AR Path="/5DC58965/5DCA99D4" Ref="D15"  Part="1"
 AR Path="/5D399F3E/5DCA99D4" Ref="D17"  Part="1"
-F 0 "D15" V 4554 3729 50  0000 L CNN
+F 0 "D17" V 4554 3729 50  0000 L CNN
 F 1 "3.6v" V 4645 3729 50  0000 L CNN
 F 2 "_Generic:SOD-523_DIODE" H 4600 3650 50  0001 C CNN
@@
 AR Path="/5DC58965/5DB5A876" Ref="Q14"  Part="1"
 AR Path="/5D399F3E/5DB5A876" Ref="Q16"  Part="1"
-F 0 "Q14" V 5700 3750 50  0000 C CNN
+F 0 "Q16" V 5700 3750 50  0000 C CNN
 F 1 "AO3402" V 5791 3750 50  0000 C CNN
 F 2 "_Generic:SOT-23" H 5650 3850 50  0001 C CNN
@@
 AR Path="/5DC58965/5DCA99D6" Ref="#PWR0195"  Part="1"
 AR Path="/5D399F3E/5DCA99D6" Ref="#PWR0206"  Part="1"
-F 0 "#PWR0195" H 6100 3650 50  0001 C CNN
+F 0 "#PWR0206" H 6100 3650 50  0001 C CNN
 F 1 "GND" H 6100 3750 50  0001 C CNN
 F 2 "" H 6100 3900 50  0001 C CNN
@@
 AR Path="/5DC58965/5DCA99D7" Ref="#PWR0196"  Part="1"
 AR Path="/5D399F3E/5DCA99D7" Ref="#PWR0207"  Part="1"
-F 0 "#PWR0196" H 6650 2950 50  0001 C CNN
+F 0 "#PWR0207" H 6650 2950 50  0001 C CNN
 F 1 "+24V" H 6665 3273 50  0000 C CNN
 F 2 "" H 6650 3100 50  0001 C CNN
@@
 AR Path="/5DC58965/5DB5A88C" Ref="#PWR0197"  Part="1"
 AR Path="/5D399F3E/5DB5A88C" Ref="#PWR0208"  Part="1"
-F 0 "#PWR0197" H 5000 3650 50  0001 C CNN
+F 0 "#PWR0208" H 5000 3650 50  0001 C CNN
 F 1 "GND" H 5000 3750 50  0001 C CNN
 F 2 "" H 5000 3900 50  0001 C CNN
@@
 AR Path="/5DC58965/5DCA99D9" Ref="C75"  Part="1"
 AR Path="/5D399F3E/5DCA99D9" Ref="C77"  Part="1"
-F 0 "C75" H 6192 3646 50  0000 L CNN
+F 0 "C77" H 6192 3646 50  0000 L CNN
 F 1 "4.7u" H 6192 3555 50  0000 L CNN
 F 2 "_Generic:0805_CAP" H 6100 3600 50  0001 C CNN
@@
 AR Path="/5DC58965/5DCA99DA" Ref="R52"  Part="1"
 AR Path="/5D399F3E/5DCA99DA" Ref="R56"  Part="1"
-F 0 "R52" H 4930 3696 50  0000 R CNN
+F 0 "R56" H 4930 3696 50  0000 R CNN
 F 1 "1meg" H 4930 3605 50  0000 R CNN
 F 2 "_Generic:0603_RES" V 4930 3650 50  0001 C CNN
@@
 AR Path="/5DC58965/5DB5A8A0" Ref="R51"  Part="1"
 AR Path="/5D399F3E/5DB5A8A0" Ref="R55"  Part="1"
-F 0 "R51" V 5207 3150 50  0000 C CNN
+F 0 "R55" V 5207 3150 50  0000 C CNN
 F 1 "4.7k" V 5116 3150 50  0000 C CNN
 F 2 "_Generic:0603_RES" V 4930 3150 50  0001 C CNN

Commit message: pcb v1
Changed lines of the file:
@@
 $Descr A4 11693 8268
 encoding utf-8
-Sheet 19 19
+Sheet 16 19
 Title ""
 Date ""
@@
 AR Path="/5DC58965/5DB5A825" Ref="J21"  Part="1"
 AR Path="/5D399F3E/5DB5A825" Ref="J23"  Part="1"
-F 0 "J23" H 6730 3792 50  0000 L CNN
+F 0 "J20" H 6730 3792 50  0000 L CNN
 F 1 "Conn_01x03" H 6730 3701 50  0001 L CNN
 F 2 "_Generic:JST_XH_3P" H 6650 3750 50  0001 C CNN
@@
 AR Path="/5DC58965/5DB5A832" Ref="JP33"  Part="1"
 AR Path="/5D399F3E/5DB5A832" Ref="JP39"  Part="1"
-F 0 "JP39" H 6558 3300 50  0000 L CNN
+F 0 "JP30" H 6558 3300 50  0000 L CNN
 F 1 "SolderJumper_4_Open" H 6400 3300 50  0001 C CNN
 F 2 "_Generic:SolderJumper_JST" H 6400 3300 50  0001 C CNN
@@
 AR Path="/5DC58965/5DCA99D2" Ref="JP31"  Part="1"
 AR Path="/5D399F3E/5DCA99D2" Ref="JP37"  Part="1"
-F 0 "JP37" V 5450 3368 50  0000 L CNN
+F 0 "JP28" V 5450 3368 50  0000 L CNN
 F 1 "SolderJumper_2_Open" H 5450 3300 50  0001 C CNN
 F 2 "_Generic:Solder Jumper 2P" H 5450 3300 50  0001 C CNN
@@
 AR Path="/5DC58965/5DCA99D3" Ref="JP32"  Part="1"
 AR Path="/5D399F3E/5DCA99D3" Ref="JP38"  Part="1"
-F 0 "JP38" V 5800 3232 50  0000 R CNN
+F 0 "JP29" V 5800 3232 50  0000 R CNN
 F 1 "SolderJumper_2_Open" H 5800 3300 50  0001 C CNN
 F 2 "_Generic:Solder Jumper 2P" H 5800 3300 50  0001 C CNN
@@
 AR Path="/5DC58965/5DCA99D4" Ref="D15"  Part="1"
 AR Path="/5D399F3E/5DCA99D4" Ref="D17"  Part="1"
-F 0 "D17" V 4554 3729 50  0000 L CNN
+F 0 "D14" V 4554 3729 50  0000 L CNN
 F 1 "3.6v" V 4645 3729 50  0000 L CNN
 F 2 "_Generic:SOD-523_DIODE" H 4600 3650 50  0001 C CNN
@@
 AR Path="/5DC58965/5DB5A876" Ref="Q14"  Part="1"
 AR Path="/5D399F3E/5DB5A876" Ref="Q16"  Part="1"
-F 0 "Q16" V 5700 3750 50  0000 C CNN
+F 0 "Q13" V 5700 3750 50  0000 C CNN
 F 1 "AO3402" V 5791 3750 50  0000 C CNN
 F 2 "_Generic:SOT-23" H 5650 3850 50  0001 C CNN
@@
 AR Path="/5DC58965/5DCA99D9" Ref="C75"  Part="1"
 AR Path="/5D399F3E/5DCA99D9" Ref="C77"  Part="1"
-F 0 "C77" H 6192 3646 50  0000 L CNN
+F 0 "C74" H 6192 3646 50  0000 L CNN
 F 1 "4.7u" H 6192 3555 50  0000 L CNN
 F 2 "_Generic:0805_CAP" H 6100 3600 50  0001 C CNN
@@
 AR Path="/5DC58965/5DCA99DA" Ref="R52"  Part="1"
 AR Path="/5D399F3E/5DCA99DA" Ref="R56"  Part="1"
-F 0 "R56" H 4930 3696 50  0000 R CNN
+F 0 "R49" H 4930 3696 50  0000 R CNN
 F 1 "1meg" H 4930 3605 50  0000 R CNN
 F 2 "_Generic:0603_RES" V 4930 3650 50  0001 C CNN
@@
 AR Path="/5DC58965/5DB5A8A0" Ref="R51"  Part="1"
 AR Path="/5D399F3E/5DB5A8A0" Ref="R55"  Part="1"
-F 0 "R55" V 5207 3150 50  0000 C CNN
+F 0 "R47" V 5207 3150 50  0000 C CNN
 F 1 "4.7k" V 5116 3150 50  0000 C CNN
 F 2 "_Generic:0603_RES" V 4930 3150 50  0001 C CNN
