File: hardware/power.sch (KiCad schematic (older format))
At the start: 76 parts, among them J100 Conn_01x01, J101 Conn_01x01, J102 Conn_01x01, J39 Screw_Terminal_01x02, J44 Conn_01x01, J45 Conn_01x01, J48 Conn_01x01, J49 Conn_01x01, J50 Conn_01x01, J51 Conn_01x01, J53 Conn_01x01, J54 Conn_01x01, J55 Conn_01x01, J56 Conn_01x01, J57 Conn_01x01, J58 Conn_01x01, J59 Conn_01x01, J68 Conn_01x01, J69 Conn_01x01, J70 Conn_01x01, J94 Conn_01x01, J95 Conn_01x01, J96 Conn_01x01, J98 Conn_01x01, J99 Conn_01x01, Q1 AON7418, U2 LM1117-3.3, U3 SY8303, U4 SY8303

Commit message: pcb v1
Parts:
- removed J100, J101, J102, J44, J50, J51, J53, J54, J55, J68, J69, J70, J96, J98, J99: Conn_01x01, _Generic:PinHeader_2.54mm_1P, symbol #Connector:Conn_01x01
- removed U2: LM1117-3.3, Package_TO_SOT_SMD:SOT-223-3_TabPin2, symbol Regulator_Linear:LM1117-3.3
- added U2: SE5218ALG-LF, Package_TO_SOT_SMD:SOT-23-5, symbol Regulator_Linear:MIC5219-3.3YM5
Connections:
- net +3V3: now also U2.5 (OUT)
- net GND: now also U2.2 (GND); no longer H1.1
- net at C20.1, L1.2: now also U2.1 (IN), U2.3 (EN)
- no-connect marks 0 -> 2
