File: hardware/c3dpb.sch (KiCad schematic (older format))
At the start: 39 parts, among them J1 Conn_01x01, J2 Conn_01x01, J24 Conn_01x01, J3 Conn_01x01, J4 Conn_01x01, J5 Conn_01x01, J6 Conn_01x01, SW1 3x6mm, SW2 3x6mm, U1 ATSAMD51J19A-M

Commit message: combine
Parts:
- removed C15, C16: 100n, _Generic:0603_CAP, symbol Device:C_Small
- removed C17: 10u, _Generic:0603_CAP, symbol Device:C_Small
- removed R2: 10k, _Generic:0603_RES, symbol Device:R
- removed R3, R4, R5: 1k, _Generic:0603_RES, symbol Device:R
- removed R6, R7: 2.2R, _Generic:0603_RES, symbol Device:R
- removed SW2: 3x6mm, _Generic:Switch_3x4mm, symbol Switch:SW_Push
Connections:
- net labels removed: ISP_BOOT, VDDA, VREFN, VREFP, VSSA
- wire segments 222 -> 196

Commit message: new con
Connections:
- wire segments 196 -> 186
Other:
- moved on the sheet: C1, R1, SW1
Changed lines of the file:
@@
 $Descr A4 11693 8268
 encoding utf-8
-Sheet 1 8
+Sheet 1 17
 Title "Kajikia - Main Sheet"
 Date "2019-01-23"
@@
 S 700  2650 650  2500
 U 5C3B9892
-F0 "Interfaces" 50
-F1 "interface.sch" 50
+F0 "Peripherals" 50
+F1 "peripheral.sch" 50
 F2 "USB_D+" B R 1350 4450 50
 F3 "USB_D-" B R 1350 4550 50
@@
 L Switch:SW_Push SW1
 U 1 1 5DDFFC25
-P 3150 7300
-F 0 "SW1" V 3104 7448 50  0000 L CNN
-F 1 "3x6mm" V 3195 7448 50  0000 L CNN
-F 2 "_Generic:Switch_3x4mm" H 3150 7500 50  0001 C CNN
-F 3 "" H 3150 7500 50  0001 C CNN
-	1    3150 7300
+P 3100 7200
+F 0 "SW1" V 3054 7348 50  0000 L CNN
+F 1 "3x6mm" V 3145 7348 50  0000 L CNN
+F 2 "_Generic:Switch_3x4mm" H 3100 7400 50  0001 C CNN
+F 3 "" H 3100 7400 50  0001 C CNN
+	1    3100 7200
 	0    1    1    0
 $EndComp
@@
 L #Power:GND #PWR02
 U 1 1 5DE40D11
-P 3150 7600
-F 0 "#PWR02" H 3150 7350 50  0001 C CNN
-F 1 "GND" H 3150 7450 50  0001 C CNN
-F 2 "" H 3150 7600 50  0001 C CNN
-F 3 "" H 3150 7600 50  0001 C CNN
-	1    3150 7600
+P 3100 7500
+F 0 "#PWR02" H 3100 7250 50  0001 C CNN
+F 1 "GND" H 3100 7350 50  0001 C CNN
+F 2 "" H 3100 7500 50  0001 C CNN
+F 3 "" H 3100 7500 50  0001 C CNN
+	1    3100 7500
 	1    0    0    -1
 $EndComp
@@
 L Device:R R1
 U 1 1 5DE81BC8
-P 3150 6850
-F 0 "R1" H 3220 6896 50  0000 L CNN
-F 1 "10k" H 3220 6805 50  0000 L CNN
-F 2 "_Generic:0603_RES" V 3080 6850 50  0001 C CNN
-F 3 "~" H 3150 6850 50  0001 C CNN
-	1    3150 6850
+P 3100 6750
+F 0 "R1" H 3170 6796 50  0000 L CNN
+F 1 "10k" H 3170 6705 50  0000 L CNN
+F 2 "_Generic:0603_RES" V 3030 6750 50  0001 C CNN
+F 3 "~" H 3100 6750 50  0001 C CNN
+	1    3100 6750
 	1    0    0    -1
 $EndComp
@@
 L Device:C_Small C1
 U 1 1 5DE81E0E
-P 3650 7300
-F 0 "C1" H 3742 7346 50  0000 L CNN
-F 1 "100n" H 3742 7255 50  0000 L CNN
-F 2 "_Generic:0603_CAP" H 3650 7300 50  0001 C CNN
-F 3 "~" H 3650 7300 50  0001 C CNN
-	1    3650 7300
-	1    0    0    -1
-$EndComp
-Wire Wire Line
-	3650 7400 3650 7550
-Wire Wire Line
-	3650 7550 3150 7550
-Wire Wire Line
-	3150 7550 3150 7500
-Wire Wire Line
-	3150 7600 3150 7550
-Connection ~ 3150 7550
-Wire Wire Line
-	3150 7100 3150 7050
-Wire Wire Line
-	3150 7050 3650 7050
-Wire Wire Line
-	3650 7050 3650 7200
-Connection ~ 3150 7050
-Wire Wire Line
-	3150 7050 3150 7000
+P 3600 7200
+F 0 "C1" H 3692 7246 50  0000 L CNN
+F 1 "100n" H 3692 7155 50  0000 L CNN
+F 2 "_Generic:0603_CAP" H 3600 7200 50  0001 C CNN
+F 3 "~" H 3600 7200 50  0001 C CNN
+	1    3600 7200
+	1    0    0    -1
+$EndComp
+Wire Wire Line
+	3600 7300 3600 7450
+Wire Wire Line
+	3600 7450 3100 7450
+Wire Wire Line
+	3100 7450 3100 7400
+Wire Wire Line
+	3100 7500 3100 7450
+Connection ~ 3100 7450
+Wire Wire Line
+	3100 7000 3100 6950
+Wire Wire Line
+	3100 6950 3600 6950
+Wire Wire Line
+	3600 6950 3600 7100
+Connection ~ 3100 6950
+Wire Wire Line
+	3100 6950 3100 6900
 $Comp
 L power:+3.3V #PWR01
 U 1 1 5DF0847B
-P 3150 6650
-F 0 "#PWR01" H 3150 6500 50  0001 C CNN
-F 1 "+3.3V" H 3165 6823 50  0000 C CNN
-F 2 "" H 3150 6650 50  0001 C CNN
-F 3 "" H 3150 6650 50  0001 C CNN
-	1    3150 6650
-	1    0    0    -1
-$EndComp
-Text Label 3650 7050 2    50   ~ 0
+P 3100 6550
+F 0 "#PWR01" H 3100 6400 50  0001 C CNN
+F 1 "+3.3V" H 3115 6723 50  0000 C CNN
+F 2 "" H 3100 6550 50  0001 C CNN
+F 3 "" H 3100 6550 50  0001 C CNN
+	1    3100 6550
+	1    0    0    -1
+$EndComp
+Text Label 3600 6950 2    50   ~ 0
 RST
 $Comp
@@
 Wire Wire Line
 	1350 4450 1850 4450
-$Sheet
-S 700  6300 650  1200
-U 606BF39C
-F0 "Power Outputs" 50
-F1 "output.sch" 50
-F2 "POWER_OUT1" I R 1350 7300 50
-F3 "POWER_OUT2" I R 1350 7400 50
-F4 "HV_IO2" B R 1350 6500 50
-F5 "HV_IO7" B R 1350 7000 50
-F6 "HV_IO8" B R 1350 7100 50
-F7 "HV_IO1" B R 1350 6400 50
-F8 "HV_IO3" B R 1350 6600 50
-F9 "HV_IO4" B R 1350 6700 50
-F10 "HV_IO5" B R 1350 6800 50
-F11 "HV_IO6" B R 1350 6900 50
-$EndSheet
-Text Label 1850 7000 2    50   ~ 0
-P1.18_ADV
-Text Label 1850 7100 2    50   ~ 0
-P1.19_ADV
-Wire Wire Line
-	1850 7100 1350 7100
-Wire Wire Line
-	1350 7000 1850 7000
-Text Label 1850 6400 2    50   ~ 0
-P0.22_ADV
-Text Label 1850 6500 2    50   ~ 0
-P1.22_ADV
-Text Label 1850 6600 2    50   ~ 0
-P1.25_ADV
-Text Label 1850 6700 2    50   ~ 0
-P1.26_ADV
-Text Label 1850 6800 2    50   ~ 0
-P1.28_ADV
-Text Label 1850 6900 2    50   ~ 0
-P1.29_ADV
-Text Label 1850 7300 2    50   ~ 0
-P2.3_POW
-Text Label 1850 7400 2    50   ~ 0
-P2.4_POW
-Wire Wire Line
-	1850 7400 1350 7400
-Wire Wire Line
-	1350 7300 1850 7300
-Wire Wire Line
-	1850 6900 1350 6900
-Wire Wire Line
-	1350 6800 1850 6800
-Wire Wire Line
-	1850 6700 1350 6700
-Wire Wire Line
-	1350 6600 1850 6600
-Wire Wire Line
-	1850 6500 1350 6500
-Wire Wire Line
-	1350 6400 1850 6400
 Text Label 9650 1400 0    50   ~ 0
 DRV1_EN
@@
 Text Notes 2600 750  0    100  ~ 20
 Processor
-Text Notes 550  6050 0    100  ~ 20
+Text Notes 550  5650 0    100  ~ 20
 Power Outputs
 Text Notes 9100 750  0    100  ~ 20
 Stepper Driver
 Wire Wire Line
-	3150 6650 3150 6700
+	3100 6550 3100 6600
 $Comp
 L Device:C_Small C31
@@
 Wire Wire Line
 	4350 4950 3850 4950
+$Sheet
+S 1550 5850 550  200
+U 5DB36909
+F0 "IO1" 50
+F1 "io.sch" 50
+F2 "IO" B R 2100 5950 50
+$EndSheet
+$Sheet
+S 1550 6250 550  200
+U 5DBDF367
+F0 "IO2" 50
+F1 "io.sch" 50
+F2 "IO" B R 2100 6350 50
+$EndSheet
+$Sheet
+S 1550 6650 550  200
+U 5DBEB073
+F0 "IO3" 50
+F1 "io.sch" 50
+F2 "IO" B R 2100 6750 50
+$EndSheet
+$Sheet
+S 1550 7050 550  200
+U 5DBF6D6B
+F0 "IO4" 50
+F1 "io.sch" 50
+F2 "IO" B R 2100 7150 50
+$EndSheet
+$Sheet
+S 1550 7450 550  200
+U 5DC02A6B
+F0 "IO5" 50
+F1 "io.sch" 50
+F2 "IO" B R 2100 7550 50
+$EndSheet
+$Sheet
+S 950  5850 550  200
+U 5DC28D35
+F0 "IO6" 50
+F1 "io_rev.sch" 50
+F2 "IO" B L 950 5950 50
+$EndSheet
+$Sheet
+S 950  6250 550  200
+U 5DC34FAD
+F0 "IO7" 50
+F1 "io_rev.sch" 50
+F2 "IO" B L 950 6350 50
+$EndSheet
+$Sheet
+S 950  6650 550  200
+U 5DC40D95
+F0 "IO8" 50
+F1 "io_rev.sch" 50
+F2 "IO" B L 950 6750 50
+$EndSheet
+$Sheet
+S 950  7050 550  200
+U 5DC4CB7D
+F0 "IO9" 50
+F1 "io_rev.sch" 50
+F2 "IO" B L 950 7150 50
+$EndSheet
+$Sheet
+S 950  7450 550  200
+U 5DC58965
+F0 "IO10" 50
+F1 "io_rev.sch" 50
+F2 "IO" B L 950 7550 50
+$EndSheet
 $EndSCHEMATC

Commit message: new con
Changed lines of the file:
@@
 $Descr A4 11693 8268
 encoding utf-8
-Sheet 1 17
+Sheet 1 19
 Title "Kajikia - Main Sheet"
 Date "2019-01-23"
@@
 $EndSheet
 $Sheet
+S 950  6250 550  200
+U 5DC28D35
+F0 "IO8" 50
+F1 "io_rev.sch" 50
+F2 "IO" B L 950 6350 50
+$EndSheet
+$Sheet
+S 950  6650 550  200
+U 5DC34FAD
+F0 "IO9" 50
+F1 "io_rev.sch" 50
+F2 "IO" B L 950 6750 50
+$EndSheet
+$Sheet
+S 950  7050 550  200
+U 5DC40D95
+F0 "IO10" 50
+F1 "io_rev.sch" 50
+F2 "IO" B L 950 7150 50
+$EndSheet
+$Sheet
+S 950  7850 550  200
+U 5DC4CB7D
+F0 "IO12" 50
+F1 "io_rev.sch" 50
+F2 "IO" B L 950 7950 50
+$EndSheet
+$Sheet
+S 950  7450 550  200
+U 5DC58965
+F0 "IO11" 50
+F1 "io_rev.sch" 50
+F2 "IO" B L 950 7550 50
+$EndSheet
+$Sheet
+S 1550 7850 550  200
+U 5D38DAD4
+F0 "IO6" 50
+F1 "io.sch" 50
+F2 "IO" B R 2100 7950 50
+$EndSheet
+$Sheet
 S 950  5850 550  200
-U 5DC28D35
-F0 "IO6" 50
+U 5D399F3E
+F0 "IO7" 50
 F1 "io_rev.sch" 50
 F2 "IO" B L 950 5950 50
 $EndSheet
-$Sheet
-S 950  6250 550  200
-U 5DC34FAD
-F0 "IO7" 50
-F1 "io_rev.sch" 50
-F2 "IO" B L 950 6350 50
-$EndSheet
-$Sheet
-S 950  6650 550  200
-U 5DC40D95
-F0 "IO8" 50
-F1 "io_rev.sch" 50
-F2 "IO" B L 950 6750 50
-$EndSheet
-$Sheet
-S 950  7050 550  200
-U 5DC4CB7D
-F0 "IO9" 50
-F1 "io_rev.sch" 50
-F2 "IO" B L 950 7150 50
-$EndSheet
-$Sheet
-S 950  7450 550  200
-U 5DC58965
-F0 "IO10" 50
-F1 "io_rev.sch" 50
-F2 "IO" B L 950 7550 50
-$EndSheet
 $EndSCHEMATC

Commit message: routing
Changed lines of the file:
@@
 $EndSheet
 $Sheet
-S 700  2650 650  2500
+S 850  2300 650  2500
 U 5C3B9892
 F0 "Peripherals" 50
 F1 "peripheral.sch" 50
-F2 "USB_D+" B R 1350 4450 50
-F3 "USB_D-" B R 1350 4550 50
-F4 "ENDSTOP1" O R 1350 2750 50
-F5 "ENDSTOP2" O R 1350 2850 50
-F6 "ENDSTOP3" O R 1350 2950 50
-F7 "ENDSTOP4" O R 1350 3050 50
-F8 "THERMISTOR1" O R 1350 3250 50
-F9 "THERMISTOR2" O R 1350 3350 50
-F10 "THERMISTOR3" O R 1350 3450 50
-F11 "THERMISTOR4" O R 1350 3550 50
-F12 "MAX_SCK" I R 1350 4750 50
-F13 "MAX_MISO" O R 1350 4850 50
-F14 "MAX_CS" I R 1350 4950 50
-F15 "BUZZER" I R 1350 3950 50
+F2 "USB_D+" B R 1500 4100 50
+F3 "USB_D-" B R 1500 4200 50
+F4 "ENDSTOP1" O R 1500 2400 50
+F5 "ENDSTOP2" O R 1500 2500 50
+F6 "ENDSTOP3" O R 1500 2600 50
+F7 "ENDSTOP4" O R 1500 2700 50
+F8 "THERMISTOR1" O R 1500 2900 50
+F9 "THERMISTOR2" O R 1500 3000 50
+F10 "THERMISTOR3" O R 1500 3100 50
+F11 "THERMISTOR4" O R 1500 3200 50
+F12 "MAX_SCK" I R 1500 4400 50
+F13 "MAX_MISO" O R 1500 4500 50
+F14 "MAX_CS" I R 1500 4600 50
+F15 "BUZZER" I R 1500 3600 50
 $EndSheet
 $Comp
@@
 Wire Wire Line
 	3800 800  3800 750
-Text Label 1850 2750 2    50   ~ 0
+Text Label 2000 2400 2    50   ~ 0
 P0.0_END
-Text Label 1850 2850 2    50   ~ 0
+Text Label 2000 2500 2    50   ~ 0
 P0.1_END
-Text Label 1850 2950 2    50   ~ 0
+Text Label 2000 2600 2    50   ~ 0
 P0.19_END
-Text Label 1850 3050 2    50   ~ 0
+Text Label 2000 2700 2    50   ~ 0
 P0.20_END
-Text Label 1850 3250 2    50   ~ 0
+Text Label 2000 2900 2    50   ~ 0
 P0.23_TH0
-Text Label 1850 3350 2    50   ~ 0
+Text Label 2000 3000 2    50   ~ 0
 P0.24_TH1
-Text Label 1850 3450 2    50   ~ 0
+Text Label 2000 3100 2    50   ~ 0
 P0.25_TH2
-Text Label 1850 3550 2    50   ~ 0
+Text Label 2000 3200 2    50   ~ 0
 P0.26_TH3
 Wire Wire Line
-	1850 3050 1350 3050
-Wire Wire Line
-	1350 2950 1850 2950
-Wire Wire Line
-	1850 2850 1350 2850
-Wire Wire Line
-	1350 2750 1850 2750
-Wire Wire Line
-	1850 3250 1350 3250
-Wire Wire Line
-	1350 3350 1850 3350
-Wire Wire Line
-	1850 3450 1350 3450
-Wire Wire Line
-	1350 3550 1850 3550
-Text Label 1850 3950 2    50   ~ 0
+	2000 2700 1500 2700
+Wire Wire Line
+	1500 2600 2000 2600
+Wire Wire Line
+	2000 2500 1500 2500
+Wire Wire Line
+	1500 2400 2000 2400
+Wire Wire Line
+	2000 2900 1500 2900
+Wire Wire Line
+	1500 3000 2000 3000
+Wire Wire Line
+	2000 3100 1500 3100
+Wire Wire Line
+	1500 3200 2000 3200
+Text Label 2000 3600 2    50   ~ 0
 BUZZER
 Wire Wire Line
-	1850 3950 1350 3950
-Text Label 1850 4450 2    50   ~ 0
+	2000 3600 1500 3600
+Text Label 2000 4100 2    50   ~ 0
 USB_D+
-Text Label 1850 4550 2    50   ~ 0
+Text Label 2000 4200 2    50   ~ 0
 USB_D-
 Wire Wire Line
-	1850 4550 1350 4550
-Wire Wire Line
-	1350 4450 1850 4450
+	2000 4200 1500 4200
+Wire Wire Line
+	1500 4100 2000 4100
 Text Label 9650 1400 0    50   ~ 0
 DRV1_EN
@@
 Wire Wire Line
 	9650 1850 10150 1850
-Text Label 1850 4750 2    50   ~ 0
+Text Label 2000 4400 2    50   ~ 0
 DRV_SCK
-Text Label 1850 4850 2    50   ~ 0
+Text Label 2000 4500 2    50   ~ 0
 DRV_MISO
-Text Label 1850 4950 2    50   ~ 0
+Text Label 2000 4600 2    50   ~ 0
 MAX1_CS
 Wire Wire Line
-	1850 4850 1350 4850
-Wire Wire Line
-	1350 4750 1850 4750
+	2000 4500 1500 4500
+Wire Wire Line
+	1500 4400 2000 4400
 Wire Notes Line
 	9050 6450 9050 550
@@
 	5850 6900 5950 6900
 Wire Wire Line
-	1350 4950 1850 4950
+	1500 4600 2000 4600
 $Sheet
 S 10150 2400 550  900

Commit message: pcb v1
Parts:
- removed C31: 10u, _Generic:0603_CAP, symbol Device:C_Small
- removed JP16: SolderJumper_3_Open, _Generic:Solder Jumper 3P, symbol #PCB_Only:SolderJumper_3_Open
- removed SW1: 3x6mm, _Generic:Switch_3x4mm, symbol Switch:SW_Push
- added FB2: 220r/100mhz, _Generic:0603_IND, symbol Device:Ferrite_Bead_Small
- added J25, J26, J27, J28, J29, J30, J31, J32, J33, J34: Conn_01x01, _Generic:PinHeader_2.54mm_1P, symbol #Connector:Conn_01x01
- C13, C14: value 100n -> 10u
- C26: value 10u -> 100n
Connections:
- net labels added: DRV1_UART, DRV2_UART, DRV3_UART, DRV4_UART, I2C_SCL, I2C_SDA, IO1, IO10, IO11, IO12, IO2, IO3, IO4, IO5, IO6, IO7, IO8, IO9, POW1, POW2, SPI_CS, SPI_MISO, SPI_MOSI, SPI_SCK, TH1, TH2, TH3
- net labels removed: +5V, DRV1_EN, DRV2_EN, DRV3_EN, DRV4_EN, DRV_MISO, DRV_SCK, DRV_UART, MAX1_CS, P0.0_END, P0.19_END, P0.1_END, P0.20_END, P0.22_ADV, P0.23_TH0, P0.24_TH1, P0.25_TH2, P0.26_TH3, P1.18_ADV, P1.19_ADV, P1.22_ADV, P1.25_ADV, P1.26_ADV, P1.28_ADV, P1.29_ADV, P2.3_POW, P2.4_POW, SCL, SDA, VDDIO
- wire segments 186 -> 177
- no-connect marks 5 -> 1
Other:
- note added: "2\n3\n0\n1"
- note removed: "sercom1.0"
- note removed: "sercom1.1"
- note removed: "usb_dm"
- note removed: "usb_dp"
- moved on the sheet: C1, C10, C11, C2, C4, C6, C7, C8, C9, R10, R37, R42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

Commit message: pcb version 1.1
Parts:
- FB2: value 220r/100mhz -> 470r/100mhz
Changed lines of the file:
@@
 EESchema Schematic File Version 4
-LIBS:c3dpb-cache
-EELAYER 29 0
+EELAYER 30 0
 EELAYER END
 $Descr A4 11693 8268
@@
 Sheet 1 19
 Title "Kajikia - Main Sheet"
-Date "2019-01-23"
-Rev "1.0"
+Date "2020-02-15"
+Rev "1.1"
 Comp "Sven Wrieden"
 Comment1 ""
@@
 P 3650 1400
 F 0 "FB2" V 3413 1400 50  0000 C CNN
-F 1 "220r/100mhz" V 3504 1400 50  0000 C CNN
+F 1 "470r/100mhz" V 3504 1400 50  0000 C CNN
 F 2 "_Generic:0603_IND" V 3580 1400 50  0001 C CNN
 F 3 "~" H 3650 1400 50  0001 C CNN
@@
 Text Label 7000 2950 0    50   ~ 0
 SPI_MISO
+$Comp
+L power:PWR_FLAG #FLG0102
+U 1 1 5E6CAF71
+P 4150 1350
+F 0 "#FLG0102" H 4150 1425 50  0001 C CNN
+F 1 "PWR_FLAG" H 4150 1523 50  0000 C CNN
+F 2 "" H 4150 1350 50  0001 C CNN
+F 3 "~" H 4150 1350 50  0001 C CNN
+	1    4150 1350
+	1    0    0    -1
+$EndComp
+Wire Wire Line
+	4150 1350 4150 1400
 $EndSCHEMATC
