File: hotend_board/c3dpb.sch (KiCad schematic (older format))
At the start: 63 parts, among them J11 Conn_01x03, J2 Conn_01x08, J5 Conn_01x02, J6 Conn_01x06, J7 Conn_01x02, Q2 AON7524, U1 BME280, U2 SY8303, U3 SE5218ALG-LF, U4 STM32F042G4Ux, U5 MAX6675

Commit message: value fixes
Parts:
- C10, C22: value 10u -> 1u
- C16, C17, C3: value 22u -> 10u
Changed lines of the file:
@@
 AR Path="/5E887778" Ref="C22"  Part="1"
 F 0 "C22" H 9558 3046 50  0000 R CNN
-F 1 "10u" H 9558 2955 50  0000 R CNN
+F 1 "1u" H 9558 2955 50  0000 R CNN
 F 2 "_Generic:0603_CAP" H 9650 3000 50  0001 C CNN
 F 3 "~" H 9650 3000 50  0001 C CNN
@@
 P 9700 5200
 F 0 "C10" H 9792 5246 50  0000 L CNN
-F 1 "10u" H 9792 5155 50  0000 L CNN
+F 1 "1u" H 9792 5155 50  0000 L CNN
 F 2 "_Generic:0603_CAP" H 9700 5200 50  0001 C CNN
 F 3 "~" H 9700 5200 50  0001 C CNN
@@
 P 1700 4600
 F 0 "C16" H 1792 4646 50  0000 L CNN
-F 1 "22u" H 1792 4555 50  0000 L CNN
+F 1 "10u" H 1792 4555 50  0000 L CNN
 F 2 "_Generic:1210_CAP" H 1700 4600 50  0001 C CNN
 F 3 "~" H 1700 4600 50  0001 C CNN
@@
 P 2200 4600
 F 0 "C17" H 2292 4646 50  0000 L CNN
-F 1 "22u" H 2292 4555 50  0000 L CNN
+F 1 "10u" H 2292 4555 50  0000 L CNN
 F 2 "_Generic:1210_CAP" H 2200 4600 50  0001 C CNN
 F 3 "~" H 2200 4600 50  0001 C CNN
@@
 P 1200 1200
 F 0 "C3" H 1292 1246 50  0000 L CNN
-F 1 "22u" H 1292 1155 50  0000 L CNN
+F 1 "10u" H 1292 1155 50  0000 L CNN
 F 2 "_Generic:1210_CAP" H 1200 1200 50  0001 C CNN
 F 3 "~" H 1200 1200 50  0001 C CNN
