File: hotend_board/fandriver.sch (KiCad schematic (older format))
At the start: 9 parts, among them J1 Conn_01x02, Q1 DMN3730U

Commit message: value fixes
Parts:
- C6: value 10u -> 1u
Changed lines of the file:
@@
 AR Path="/5E9D1609/5E9F5F45" Ref="Q3"  Part="1"
 AR Path="/5E9E2ADA/5E9F5F45" Ref="Q4"  Part="1"
-F 0 "Q4" H 5154 3796 50  0000 L CNN
+F 0 "Q3" H 5154 3796 50  0000 L CNN
 F 1 "DMN3730U" H 5154 3705 50  0000 L CNN
 F 2 "_Generic:SOT-23" H 5150 3850 50  0001 C CNN
@@
 AR Path="/5E9D1609/5E986F15" Ref="#PWR022"  Part="1"
 AR Path="/5E9E2ADA/5E986F15" Ref="#PWR024"  Part="1"
-F 0 "#PWR024" H 5050 4100 50  0001 C CNN
+F 0 "#PWR022" H 5050 4100 50  0001 C CNN
 F 1 "GND" H 5050 4200 50  0001 C CNN
 F 2 "" H 5050 4350 50  0001 C CNN
@@
 AR Path="/5E9D1609/5E986F1C" Ref="R13"  Part="1"
 AR Path="/5E9E2ADA/5E986F1C" Ref="R17"  Part="1"
-F 0 "R17" H 4630 4146 50  0000 R CNN
+F 0 "R13" H 4630 4146 50  0000 R CNN
 F 1 "1meg" H 4630 4055 50  0000 R CNN
 F 2 "_Generic:0603_RES" V 4630 4100 50  0001 C CNN
@@
 AR Path="/5E9D1609/5E986F22" Ref="R12"  Part="1"
 AR Path="/5E9E2ADA/5E986F22" Ref="R16"  Part="1"
-F 0 "R16" V 4707 3750 50  0000 C CNN
+F 0 "R12" V 4707 3750 50  0000 C CNN
 F 1 "100R" V 4616 3750 50  0000 C CNN
 F 2 "_Generic:0603_RES" V 4430 3750 50  0001 C CNN
@@
 AR Path="/5E9D1609/5E986F28" Ref="J3"  Part="1"
 AR Path="/5E9E2ADA/5E986F28" Ref="J4"  Part="1"
-F 0 "J4" H 7100 3400 50  0000 C CNN
+F 0 "J3" H 7100 3400 50  0000 C CNN
 F 1 "Conn_01x02" H 7250 3300 50  0001 C CNN
 F 2 "Connector_JST:JST_SH_BM02B-SRSS-TB_1x02-1MP_P1.00mm_Vertical" H 6950 3400 50  0001 C CNN
@@
 AR Path="/5E9D1609/5E986F40" Ref="C8"  Part="1"
 AR Path="/5E9E2ADA/5E986F40" Ref="C11"  Part="1"
-F 0 "C11" H 6342 3146 50  0000 L CNN
-F 1 "10u" H 6342 3055 50  0000 L CNN
+F 0 "C8" H 6342 3146 50  0000 L CNN
+F 1 "1u" H 6342 3055 50  0000 L CNN
 F 2 "_Generic:0603_CAP" H 6250 3100 50  0001 C CNN
 F 3 "~" H 6250 3100 50  0001 C CNN
@@
 AR Path="/5E9D1609/5E986F59" Ref="R14"  Part="1"
 AR Path="/5E9E2ADA/5E986F59" Ref="R18"  Part="1"
-F 0 "R18" H 6320 3746 50  0000 L CNN
+F 0 "R14" H 6320 3746 50  0000 L CNN
 F 1 "100k" H 6320 3655 50  0000 L CNN
 F 2 "_Generic:0603_RES" V 6180 3700 50  0001 C CNN
@@
 AR Path="/5E9D1609/5E9F5F4F" Ref="R15"  Part="1"
 AR Path="/5E9E2ADA/5E9F5F4F" Ref="R19"  Part="1"
-F 0 "R19" H 6320 4146 50  0000 L CNN
+F 0 "R15" H 6320 4146 50  0000 L CNN
 F 1 "10k" H 6320 4055 50  0000 L CNN
 F 2 "_Generic:0603_RES" V 6180 4100 50  0001 C CNN
@@
 AR Path="/5E9D1609/5E9F5F50" Ref="#PWR011"  Part="1"
 AR Path="/5E9E2ADA/5E9F5F50" Ref="#PWR023"  Part="1"
-F 0 "#PWR023" H 5050 2700 50  0001 C CNN
+F 0 "#PWR011" H 5050 2700 50  0001 C CNN
 F 1 "+24V" H 5065 3023 50  0000 C CNN
 F 2 "" H 5050 2850 50  0001 C CNN
@@
 AR Path="/5E9D1609/5E986F34" Ref="L2"  Part="1"
 AR Path="/5E9E2ADA/5E986F34" Ref="L3"  Part="1"
-F 0 "L3" V 5840 3500 50  0000 C CNN
+F 0 "L2" V 5840 3500 50  0000 C CNN
 F 1 "CBC3225T221KR" V 5749 3500 50  0000 C CNN
 F 2 "_Generic:1210_CAP" H 5650 3500 50  0001 C CNN
@@
 AR Path="/5E9D1609/5E986F2E" Ref="D6"  Part="1"
 AR Path="/5E9E2ADA/5E986F2E" Ref="D7"  Part="1"
-F 0 "D7" V 5004 3179 50  0000 L CNN
+F 0 "D6" V 5004 3179 50  0000 L CNN
 F 1 "MSK4010" V 5095 3179 50  0000 L CNN
 F 2 "_Generic:SOD-523_DIODE" H 5050 3100 50  0001 C CNN
@@
 AR Path="/5E9D1609/5F780CE3" Ref="#PWR0121"  Part="1"
 AR Path="/5E9E2ADA/5F780CE3" Ref="#PWR0122"  Part="1"
-F 0 "#PWR0122" H 7350 3550 50  0001 C CNN
+F 0 "#PWR0121" H 7350 3550 50  0001 C CNN
 F 1 "+24V" H 7365 3873 50  0000 C CNN
 F 2 "" H 7350 3700 50  0001 C CNN
