File: hotend_board/c3dpb.kicad_pcb (KiCad board)
At the start: 2 copper layers, 30 x 20 mm, 87 parts, among them J1 Conn_01x02, J11 Conn_01x03, J2 Conn_01x08, J3 Conn_01x02, J4 Conn_01x02, J5 Conn_01x02, J6 Conn_01x06, J7 Conn_01x02, Q1 DMN3730U, Q2 AON7524, Q3 DMN3730U, Q4 DMN3730U, U1 BME280, U2 SY8303, U3 SE5218ALG-LF, U4 STM32F042G4Ux, U5 MAX6675

Commit message: hotend board v1.0
Parts:
- removed C12: 22u, _Generic:1210_CAP
- added C13: 10u, _Generic:0603_CAP, B.Cu at (96.2, 79.2)
- added C2: 10u, _Generic:0603_CAP, B.Cu at (97.8, 82.0)
- added C24: 10u, _Generic:0603_CAP, B.Cu at (96.2, 82.0)
- added C7: 10u, _Generic:0603_CAP, B.Cu at (97.8, 79.2)
Routing:
- net +5V: track 41.8 -> 35.3 mm
- net GND: track 158.0 -> 160.8 mm, vias 34 -> 39

Commit message: idk backup...
Parts:
- C10, C11, C22, C6, C8: value 10u -> 1u
- C16, C17, C3: value 22u -> 10u
